Commit message: Update car.xacro add transmission tag to all joints which are children of controllable joints

File: 3_control/car_description/urdf/car.xacro (robot description, xacro)
@@ -69,5 +69,5 @@
 	    		</inertial>
 	 	</link>
-	<link name ="chassis">
+	<link name ="chassis"> <!--The mesh of the car -->
 		<visual>
 				<geometry>
@@ -79,5 +79,5 @@
 				<origin rpy="0 0 0" xyz="0 0 ${radius_wheel}"/>
 				<geometry>
-	       				<box size="${base_x_size} ${base_y_size} ${base_z_size}"/>
+	       				<box size="0.001 0.001 0.001"/>
 				</geometry>
 			</collision>
@@ -313,4 +313,23 @@
     </joint>
     </transmission>
+ <!-- transmission for non controllable joints-->
+   <transmission name="Front_left_wheel_controller">
+    <type>transmission_interface/SimpleTransmission</type>
+    <actuator name="motor6">
+      <mechanicalReduction>0</mechanicalReduction>
+    </actuator>
+    <joint name="Front_left_wheel_joint">
+      <hardwareInterface>hardware_interface/EffortJointInterface</hardwareInterface>
+    </joint>
+    </transmission>
+   <transmission name="Front_right_wheel_controller">
+    <type>transmission_interface/SimpleTransmission</type>
+    <actuator name="motor7">
+      <mechanicalReduction>0</mechanicalReduction>
+    </actuator>
+    <joint name="Front_right_wheel_joint">
+      <hardwareInterface>hardware_interface/EffortJointInterface</hardwareInterface>
+    </joint>
+    </transmission>
 <!--SENSORS -->
 <!-- Camera joint -->

Commit message: Change laser's position in car.xacro

File: 3_control/car_description/urdf/car.xacro (robot description, xacro)
@@ -365,5 +365,5 @@
   <!-- Hokuyo joint -->
   <joint name="hokuyo_joint" type="fixed">
-    <origin xyz="1.050 -0.2 0.5" rpy="0 0 0"/>
+    <origin xyz="1.07 -0.2 0.0" rpy="0 0 0"/>
     <parent link="base_link"/>
     <axis xyz="0 1 0" />

Commit message: Fix footprint in teb_local_planner_params and change laser's position

File: 3_control/car_description/urdf/car.xacro (robot description, xacro)
@@ -365,5 +365,5 @@
   <!-- Hokuyo joint -->
   <joint name="hokuyo_joint" type="fixed">
-    <origin xyz="1.07 -0.2 0.0" rpy="0 0 0"/>
+    <origin xyz="1.8 0.0 0.0" rpy="0 0 0"/> <!-- 1.07 -0.2 -->
     <parent link="base_link"/>
     <axis xyz="0 1 0" />

Commit message: change roscontrol plugin from .xarco to .gazebo

File: 3_control/car_description/urdf/car.xacro (robot description, xacro)
@@ -6,10 +6,10 @@
 	name="robot1_xacro">
 	<!-- Car properties !!! Y is forward-->
-	<xacro:property name="base_mass" value="5" /> <!-- in kg-->
+	<xacro:property name="base_mass" value="20" /> <!-- in kg-->
 	<xacro:property name="base_x_size" value="2.130" /> 	<!-- x is mhkos forward -->
   	<xacro:property name="base_y_size" value="0.8935" /> 	<!-- y is platos -->
   	<xacro:property name="base_z_size" value="0.1" /><!-- z is ipsos -->
 	<!-- Wheels -->
-	<xacro:property name="wheel_mass" value="1" /> <!-- in kg-->
+	<xacro:property name="wheel_mass" value="2" /> <!-- in kg-->
 	<xacro:property name="length_wheel" value="0.190" />
 	<xacro:property name="radius_wheel" value="0.261" />
@@ -267,13 +267,4 @@
    <origin rpy="0 0 0" xyz="0 0 0"/>
  </joint>
-<!-- ROS Control plugin for Gazebo -->
-  <gazebo>
-<static>false</static>
-    <plugin name="gazebo_ros_control" filename="libgazebo_ros_control.so">
-      <robotNamespace>/car</robotNamespace>
-	<robotSimType>gazebo_ros_control/DefaultRobotHWSim</robotSimType>
-	<legacyModeNS>false</legacyModeNS>
-    </plugin>
-  </gazebo>
  <!-- transmission -->
   <transmission name="Turner_right_position_controller">

Commit message: Odometry.py is no longer used the robot uses p3d_base_controller(robot.gazebo) change cars weight and add some comments (car.xarco)

File: 3_control/car_description/urdf/car.xacro (robot description, xacro)
@@ -28,5 +28,5 @@
 	              izz="${m*r*r/2}" />
 	</macro>
-	<link name="base_footprint">
+	<link name="base_footprint">  <!-- used because KDL doesnt not support a root link with an inertia -->
    		<visual>
 			<geometry>
