Commit message: Add robot_localization

File: 0_frt_common/robot/urdf/robot.xacro (robot description, xacro)
@@ -178,5 +178,5 @@
    	<origin rpy="-1.5707 0 0" xyz="-0.1 -0.15 0"/>
 	</joint>
-  <!-- Camera joint
+  <!-- Camera joint -->
   <joint name="camera_joint" type="fixed">
     <axis xyz="0 1 0" />
@@ -184,6 +184,6 @@
     <parent link="base_link"/>
     <child link="camera_link"/>
-  </joint> -->
-  <!-- Camera
+  </joint>
+  <!-- Camera -->
   <link name="camera_link">
     <collision>
@@ -207,5 +207,5 @@
       <inertia ixx="1e-6" ixy="0" ixz="0" iyy="1e-6" iyz="0" izz="1e-6" />
     </inertial>
-  </link> -->
+  </link>
   <!-- Hokuyo joint -->
   <joint name="hokuyo_joint" type="fixed">
@@ -236,19 +236,20 @@
   </link>
   <!-- Drive controller -->
-<gazebo>
-  <plugin name="skid_steer_drive_controller" filename="libgazebo_ros_skid_steer_drive.so">
-    <updateRate>100.0</updateRate>
-    <robotNamespace>/</robotNamespace>
-    <leftFrontJoint>base_to_wheel1</leftFrontJoint>
-    <rightFrontJoint>base_to_wheel3</rightFrontJoint>
-    <leftRearJoint>base_to_wheel2</leftRearJoint>
-    <rightRearJoint>base_to_wheel4</rightRearJoint>
-    <wheelSeparation>4</wheelSeparation>
-    <wheelDiameter>0.1</wheelDiameter>
-    <robotBaseFrame>base_footprint</robotBaseFrame>
-    <torque>3</torque>
-    <topicName>cmd_vel</topicName>
-    <broadcastTF>1</broadcastTF>
-  </plugin>
-</gazebo>
+  <gazebo>
+    <plugin name="skid_steer_drive_controller" filename="libgazebo_ros_skid_steer_drive.so">
+      <updateRate>100.0</updateRate>
+      <robotNamespace>/</robotNamespace>
+      <leftFrontJoint>base_to_wheel1</leftFrontJoint>
+      <rightFrontJoint>base_to_wheel3</rightFrontJoint>
+      <leftRearJoint>base_to_wheel2</leftRearJoint>
+      <rightRearJoint>base_to_wheel4</rightRearJoint>
+      <wheelSeparation>4</wheelSeparation>
+      <wheelDiameter>0.1</wheelDiameter>
+      <robotBaseFrame>base_footprint</robotBaseFrame>
+      <torque>3</torque>
+      <topicName>cmd_vel</topicName>
+      <broadcastTF>0</broadcastTF> <!-- se to 0 if you have your own odom -> base_link tf -->
+      <odometryTopic>controller/odom</odometryTopic>
+    </plugin>
+  </gazebo>
 </robot>

Commit message: Add imu to robot

File: 0_frt_common/robot/urdf/robot.xacro (robot description, xacro)
@@ -235,21 +235,30 @@
     </inertial>
   </link>
-  <!-- Drive controller -->
-  <gazebo>
-    <plugin name="skid_steer_drive_controller" filename="libgazebo_ros_skid_steer_drive.so">
-      <updateRate>100.0</updateRate>
-      <robotNamespace>/</robotNamespace>
-      <leftFrontJoint>base_to_wheel1</leftFrontJoint>
-      <rightFrontJoint>base_to_wheel3</rightFrontJoint>
-      <leftRearJoint>base_to_wheel2</leftRearJoint>
-      <rightRearJoint>base_to_wheel4</rightRearJoint>
-      <wheelSeparation>4</wheelSeparation>
-      <wheelDiameter>0.1</wheelDiameter>
-      <robotBaseFrame>base_footprint</robotBaseFrame>
-      <torque>3</torque>
-      <topicName>cmd_vel</topicName>
-      <broadcastTF>0</broadcastTF> <!-- se to 0 if you have your own odom -> base_link tf -->
-      <odometryTopic>controller/odom</odometryTopic>
-    </plugin>
-  </gazebo>
+  <!-- imu joint & link -->
+  <joint name="imu_joint" type="fixed">
+    <axis xyz="0 0 1" />
+    <origin xyz="0 0 0" rpy="0 0 0"/>
+    <parent link="base_link"/>
+    <child link="base_imu_link"/>
+  </joint>
+  <link name="base_imu_link">
+    <collision>
+      <origin xyz="0 0 0" rpy="0 0 0"/>
+      <geometry>
+        <box size="0.02 0.02 0.02"/>
+      </geometry>
+    </collision>
+    <visual>
+      <origin xyz="0 0 0" rpy="0 0 0"/>
+      <geometry>
+        <box size="0.02 0.02 0.02"/>
+      </geometry>
+      <material name="red"/>
+    </visual>
+    <inertial>
+      <mass value="0.001" />
+      <origin xyz="0 0 0" rpy="0 0 0"/>
+      <inertia ixx="0.00000015" ixy="0" ixz="0" iyy="0.00000015" iyz="0" izz="0.00000015" />
+    </inertial>
+  </link>
 </robot>

Commit message: Clean some files, update README, simulation now works but badly

File: 0_frt_common/robot/urdf/robot.xacro (robot description, xacro)
@@ -1,181 +1,181 @@
 <?xml version="1.0"?>
-<robot xmlns:xacro="http://www.ros.org/wiki/xacro"
- 	xmlns:sensor="http://playerstage.sourceforge.net/gazebo/xmlschema/#sensor"
-  xmlns:controller="http://playerstage.sourceforge.net/gazebo/xmlschema/#controller"
-  xmlns:interface="http://playerstage.sourceforge.net/gazebo/xmlschema/#interface"
-	name="robot1_xacro">
-	<xacro:property name="base_mass" value="5" /> <!-- in kg-->
-	<xacro:property name="base_x_size" value="0.2" />
+<robot  xmlns:xacro="http://www.ros.org/wiki/xacro"
+        xmlns:sensor="http://playerstage.sourceforge.net/gazebo/xmlschema/#sensor"
+        xmlns:controller="http://playerstage.sourceforge.net/gazebo/xmlschema/#controller"
+        xmlns:interface="http://playerstage.sourceforge.net/gazebo/xmlschema/#interface"
+        name="robot">
+  <xacro:property name="base_mass" value="5" /> <!-- in kg-->
+  <xacro:property name="base_x_size" value="0.2" />
   <xacro:property name="base_y_size" value="0.3" />
   <xacro:property name="base_z_size" value="0.1" />
-	<!-- Wheels -->
+  <!-- Wheels -->
   <xacro:property name="wheel_mass" value="1" /> <!-- in kg-->
-	<xacro:property name="length_wheel" value="0.05" />
-	<xacro:property name="radius_wheel" value="0.05" />
-	<xacro:property name="camera_link" value="0.05" />
-	<xacro:macro name="default_inertial" params="mass">
-  	<inertial>
-    	<mass value="${mass}" />
+  <xacro:property name="length_wheel" value="0.05" />
+  <xacro:property name="radius_wheel" value="0.05" />
+  <xacro:property name="camera_link" value="0.05" />
+  <xacro:macro name="default_inertial" params="mass">
+    <inertial>
+      <mass value="${mass}" />
       <inertia ixx="1.0" ixy="0.0" ixz="0.0" iyy="1.0" iyz="0.0" izz="1.0" />
     </inertial>
-	</xacro:macro>
-	<macro name="box_inertia" params="m x y z">
-  	<inertia  ixx="${m*(y*y+z*z)/12}" ixy = "0" ixz = "0"
-  	          iyy="${m*(x*x+z*z)/12}" iyz = "0"
-  	          izz="${m*(x*x+z*z)/12}" />
-	</macro>
-	<macro name="cylinder_inertia" params="m r h">
-		<inertia  ixx="${m*(3*r*r+h*h)/12}" ixy = "0" ixz = "0"
-	            iyy="${m*(3*r*r+h*h)/12}" iyz = "0"
-	            izz="${m*r*r/2}" />
-	</macro>
-	<link name="base_footprint">
-  	<visual>
-			<geometry>
-    		<box size="0.001 0.001 0.001"/>
-    	</geometry>
-			<origin rpy="0 0 0" xyz="0 0 0"/>
-   	</visual>
- 	</link>
- 	<xacro:include filename="$(find robot)/urdf/robot.gazebo" />
-	<gazebo reference="base_footprint">
-		<material>Gazebo/Green</material>
-		<turnGravityOff>false</turnGravityOff>
-	</gazebo>
-	<joint name="base_footprint_joint" type="fixed">
-		<origin xyz="0 0 0.15" />
-		<parent link="base_footprint" />
-		<child link="base_link" />
-	</joint>
-	<link name="base_link">
-  	<visual>
-			<geometry>
-      	<box size="${base_x_size} .3 .1"/>
-     	</geometry>
-			<origin rpy="0 0 1.54" xyz="0 0 0"/>
-			<material name="white">
-				<color rgba="1 1 1 1"/>
-			</material>
-   	</visual>
-		<collision>
-			<geometry>
-      	<box size="0.2 .3 0.1"/>
-			</geometry>
-		</collision>
-		<inertial>
-    	<mass value="${base_mass}" />
-      	<origin xyz="0 0 0" />
-      	<!--The 3x3 rotational inertia matrix. -->
-      	<box_inertia  m="${base_mass}" x="${base_x_size}" y="${base_y_size}" z="${base_z_size}"/>
-    </inertial>
- 	</link>
- 	<link name="wheel_1">
-  	<visual>
-    	<geometry>
-      	<cylinder length="${length_wheel}" radius="${radius_wheel}"/>
-     	</geometry>
-			<!-- <origin rpy="0 1.5 0" xyz="0.1 0.1 0"/> -->
-			<origin rpy="0 0 0" xyz="0 0 0"/>
-   			<material name="black">
-				<color rgba="0 0 0 1"/>
-			</material>
-		</visual>
-		<collision>
-			<geometry>
-      	<cylinder length="${length_wheel}" radius="${radius_wheel}"/>
-			</geometry>
-		</collision>
-		<inertial>
-    	<mass value="${wheel_mass}" />
-     	<origin xyz="0 0 0" />
-    	<cylinder_inertia  m="${wheel_mass}" r="${radius_wheel}" h="${length_wheel}" />
-    </inertial>
- 	</link>
- 	<link name="wheel_2">
-  	<visual>
-    	<geometry>
-      	<cylinder length="${length_wheel}" radius="${radius_wheel}"/>
-     	</geometry>
-			<!-- <origin rpy="0 1.5 0" xyz="-0.1 0.1 0"/> -->
-			<origin rpy="0 0 0" xyz="0 0 0"/>
-   			<material name="black"/>
-   	</visual>
-		<collision>
-			<geometry>
-      	<cylinder length="${length_wheel}" radius="${radius_wheel}"/>
-			</geometry>
-		</collision>
-		<inertial>
-    	<mass value="${wheel_mass}" />
-    	<origin xyz="0 0 0" />
-    	<cylinder_inertia  m="${wheel_mass}" r="${radius_wheel}" h="${length_wheel}" />
-    </inertial>
- 	</link>
- 	<link name="wheel_3">
-  	<visual>
-    	<geometry>
-      	<cylinder length="${length_wheel}" radius="${radius_wheel}"/>
-     	</geometry>
-			<!-- <origin rpy="0 1.5 0" xyz="0.1 -0.1 0"/> -->
-			<origin rpy="0 0 0" xyz="0 0 0"/>
-   			<material name="black"/>
-   	</visual>
-		<collision>
-			<geometry>
-      	<cylinder length="${length_wheel}" radius="${radius_wheel}"/>
-			</geometry>
-		</collision>
-		<inertial>
-    	<mass value="${wheel_mass}" />
-    	<origin xyz="0 0 0" />
-    	<cylinder_inertia  m="${wheel_mass}" r="${radius_wheel}" h="${length_wheel}" />
-    </inertial>
- 	</link>
- 	<link name="wheel_4">
-  	<visual>
-    	<geometry>
-      	<cylinder length="${length_wheel}" radius="${radius_wheel}"/>
-     	</geometry>
-			<!--	<origin rpy="0 1.5 0" xyz="-0.1 -0.1 0"/> -->
-			<origin rpy="0 0 0" xyz="0 0 0" />
-   			<material name="black"/>
-   	</visual>
-		<collision>
-			<geometry>
-      	<cylinder length="${length_wheel}" radius="${radius_wheel}"/>
-			</geometry>
-		</collision>
-		<inertial>
-    	<mass value="${wheel_mass}" />
-      <origin xyz="0 0 0" />
-    	<cylinder_inertia  m="${wheel_mass}" r="${radius_wheel}" h="${length_wheel}" />
-    </inertial>
- 	</link>
- 	<joint name="base_to_wheel1" type="continuous">
-   	<parent link="base_link"/>
-   	<child link="wheel_1"/>
-   	<origin rpy="-1.5707 0 0" xyz="0.1 0.15 0"/>
-   	<axis xyz="0 0 1" />
- 	</joint>
- 	<joint name="base_to_wheel2" type="continuous">
-   	<axis xyz="0 0 1" />
-   	<anchor xyz="0 0 0" />
-   	<limit effort="100" velocity="100" />
-   	<parent link="base_link"/>
-   	<child link="wheel_2"/>
-   	<origin rpy="-1.5707 0 0" xyz="-0.1 0.15 0"/>
-	</joint>
- 	<joint name="base_to_wheel3" type="continuous">
-   	<parent link="base_link"/>
-   	<axis xyz="0 0 1" />
-   	<child link="wheel_3"/>
-   	<origin rpy="-1.5707 0 0" xyz="0.1 -0.15 0"/>
- 	</joint>
- 	<joint name="base_to_wheel4" type="continuous">
-   	<parent link="base_link"/>
-   	<axis xyz="0 0 1" />
-   	<child link="wheel_4"/>
-   	<origin rpy="-1.5707 0 0" xyz="-0.1 -0.15 0"/>
-	</joint>
+  </xacro:macro>
+  <macro name="box_inertia" params="m x y z">
+    <inertia  ixx="${m*(y*y+z*z)/12}" ixy = "0" ixz = "0"
+              iyy="${m*(x*x+z*z)/12}" iyz = "0"
+              izz="${m*(x*x+z*z)/12}" />
+  </macro>
+  <macro name="cylinder_inertia" params="m r h">
+    <inertia  ixx="${m*(3*r*r+h*h)/12}" ixy = "0" ixz = "0"
+              iyy="${m*(3*r*r+h*h)/12}" iyz = "0"
+              izz="${m*r*r/2}" />
+  </macro>
+  <link name="base_footprint">
+    <visual>
+      <geometry>
+        <box size="0.001 0.001 0.001"/>
+      </geometry>
+      <origin rpy="0 0 0" xyz="0 0 0"/>
+     </visual>
+  </link>
+  <xacro:include filename="$(find robot)/urdf/robot.gazebo" />
+  <gazebo reference="base_footprint">
+    <material>Gazebo/Green</material>
+    <turnGravityOff>false</turnGravityOff>
+  </gazebo>
+  <joint name="base_footprint_joint" type="fixed">
+    <origin xyz="0 0 0.15" />
+    <parent link="base_footprint" />
+    <child link="base_link" />
+  </joint>
+  <link name="base_link">
+    <visual>
+      <geometry>
+        <box size="${base_x_size} .3 .1"/>
+      </geometry>
+      <origin rpy="0 0 1.54" xyz="0 0 0"/>
+      <material name="white">
+        <color rgba="1 1 1 1"/>
+      </material>
+    </visual>
+    <collision>
+      <geometry>
+        <box size="0.2 .3 0.1"/>
+      </geometry>
+    </collision>
+    <inertial>
+      <mass value="${base_mass}" />
+      <origin xyz="0 0 0" />
+      <!--The 3x3 rotational inertia matrix. -->
+      <box_inertia  m="${base_mass}" x="${base_x_size}" y="${base_y_size}" z="${base_z_size}"/>
+    </inertial>
+  </link>
+  <link name="wheel_1">
+    <visual>
+      <geometry>
+        <cylinder length="${length_wheel}" radius="${radius_wheel}"/>
+      </geometry>
+      <!-- <origin rpy="0 1.5 0" xyz="0.1 0.1 0"/> -->
+      <origin rpy="0 0 0" xyz="0 0 0"/>
+      <material name="black">
+        <color rgba="0 0 0 1"/>
+      </material>
+    </visual>
+    <collision>
+      <geometry>
+        <cylinder length="${length_wheel}" radius="${radius_wheel}"/>
+      </geometry>
+    </collision>
+    <inertial>
+      <mass value="${wheel_mass}" />
+       <origin xyz="0 0 0" />
+      <cylinder_inertia  m="${wheel_mass}" r="${radius_wheel}" h="${length_wheel}" />
+    </inertial>
+  </link>
+  <link name="wheel_2">
+    <visual>
+      <geometry>
+        <cylinder length="${length_wheel}" radius="${radius_wheel}"/>
+      </geometry>
+      <!-- <origin rpy="0 1.5 0" xyz="-0.1 0.1 0"/> -->
+      <origin rpy="0 0 0" xyz="0 0 0"/>
+      <material name="black"/>
+    </visual>
+    <collision>
+      <geometry>
+        <cylinder length="${length_wheel}" radius="${radius_wheel}"/>
+      </geometry>
+    </collision>
+    <inertial>
+      <mass value="${wheel_mass}" />
+      <origin xyz="0 0 0" />
+      <cylinder_inertia  m="${wheel_mass}" r="${radius_wheel}" h="${length_wheel}" />
+    </inertial>
+  </link>
+  <link name="wheel_3">
+    <visual>
+      <geometry>
+        <cylinder length="${length_wheel}" radius="${radius_wheel}"/>
+      </geometry>
+      <!-- <origin rpy="0 1.5 0" xyz="0.1 -0.1 0"/> -->
+      <origin rpy="0 0 0" xyz="0 0 0"/>
+      <material name="black"/>
+    </visual>
+    <collision>
+      <geometry>
+        <cylinder length="${length_wheel}" radius="${radius_wheel}"/>
+      </geometry>
+    </collision>
+    <inertial>
+      <mass value="${wheel_mass}" />
+      <origin xyz="0 0 0" />
+      <cylinder_inertia  m="${wheel_mass}" r="${radius_wheel}" h="${length_wheel}" />
+    </inertial>
+  </link>
+  <link name="wheel_4">
+    <visual>
+      <geometry>
+        <cylinder length="${length_wheel}" radius="${radius_wheel}"/>
+      </geometry>
+      <!--  <origin rpy="0 1.5 0" xyz="-0.1 -0.1 0"/> -->
+      <origin rpy="0 0 0" xyz="0 0 0" />
+      <material name="black"/>
+    </visual>
+    <collision>
+      <geometry>
+        <cylinder length="${length_wheel}" radius="${radius_wheel}"/>
+      </geometry>
+    </collision>
+    <inertial>
+      <mass value="${wheel_mass}" />
+      <origin xyz="0 0 0" />
+      <cylinder_inertia  m="${wheel_mass}" r="${radius_wheel}" h="${length_wheel}" />
+    </inertial>
+  </link>
+  <joint name="base_to_wheel1" type="continuous">
+    <parent link="base_link"/>
+    <child link="wheel_1"/>
+    <origin rpy="-1.5707 0 0" xyz="0.1 0.15 0"/>
+    <axis xyz="0 0 1" />
+  </joint>
+  <joint name="base_to_wheel2" type="continuous">
+    <axis xyz="0 0 1" />
+    <anchor xyz="0 0 0" />
+    <limit effort="100" velocity="100" />
+    <parent link="base_link"/>
+    <child link="wheel_2"/>
+    <origin rpy="-1.5707 0 0" xyz="-0.1 0.15 0"/>
+  </joint>
+  <joint name="base_to_wheel3" type="continuous">
+    <parent link="base_link"/>
+    <axis xyz="0 0 1" />
+    <child link="wheel_3"/>
+    <origin rpy="-1.5707 0 0" xyz="0.1 -0.15 0"/>
+  </joint>
+  <joint name="base_to_wheel4" type="continuous">
+    <parent link="base_link"/>
+    <axis xyz="0 0 1" />
+    <child link="wheel_4"/>
+    <origin rpy="-1.5707 0 0" xyz="-0.1 -0.15 0"/>
+  </joint>
   <!-- Camera joint -->
   <joint name="camera_joint" type="fixed">
@@ -190,14 +190,14 @@
       <origin xyz="0 0 0" rpy="0 0 0"/>
       <geometry>
-				<box size="0.05 0.05 0.05"/>
-      </geometry>
-    </collision>
-    <visual>
-      <origin xyz="0 0 0" rpy="0 0 0"/>
-      <geometry>
-				<box size="0.05 0.05 0.05"/>
+        <box size="0.05 0.05 0.05"/>
+      </geometry>
+    </collision>
+    <visual>
+      <origin xyz="0 0 0" rpy="0 0 0"/>
+      <geometry>
+        <box size="0.05 0.05 0.05"/>
       </geometry>
       <material name="red">
-				<color rgba="1 0 0 1"/>
+        <color rgba="1 0 0 1"/>
       </material>
     </visual>
@@ -220,5 +220,5 @@
       <origin xyz="0 0 0" rpy="0 0 0"/>
       <geometry>
-				<box size="0.01 -0.05 0.06"/>
+        <box size="0.01 -0.05 0.06"/>
       </geometry>
     </collision>
