Commit message: Clean some files, update README, simulation now works but badly

File: 3_control/car_description/urdf/car.xacro (robot description, xacro)
@@ -1,271 +1,271 @@
 <?xml version="1.0"?>
-<robot xmlns:xacro="http://www.ros.org/wiki/xacro"
- 	xmlns:sensor="http://playerstage.sourceforge.net/gazebo/xmlschema/#sensor"
-    	xmlns:controller="http://playerstage.sourceforge.net/gazebo/xmlschema/#controller"
-    	xmlns:interface="http://playerstage.sourceforge.net/gazebo/xmlschema/#interface"
-	name="robot1_xacro">
-	<!-- Car properties !!! Y is forward-->
-	<xacro:property name="base_mass" value="20" /> <!-- in kg-->
-	<xacro:property name="base_x_size" value="2.130" /> 	<!-- x is mhkos forward -->
-  	<xacro:property name="base_y_size" value="0.8935" /> 	<!-- y is platos -->
-  	<xacro:property name="base_z_size" value="0.1" /><!-- z is ipsos -->
-	<!-- Wheels -->
-	<xacro:property name="wheel_mass" value="2" /> <!-- in kg-->
-	<xacro:property name="length_wheel" value="0.190" />
-	<xacro:property name="radius_wheel" value="0.261" />
-	<!-- OFFSETS -->
-	<xacro:property name="x_offset" value="0.7625" /> <!-- metaksonio -->
-  	<xacro:property name="y_offset" value="0.5652" /> <!-- metatroxio -->
-  	<xacro:property name="z_offset" value="${radius_wheel - 0.0001}" /> <!-- diafora ipsous chassis me rodes -->
-  	<macro name="box_inertia" params="m x y z">
-  	  <inertia  ixx="${m*(y*y+z*z)/12}" ixy = "0" ixz = "0"
-  	            iyy="${m*(x*x+z*z)/12}" iyz = "0"
-  	            izz="${m*(x*x+z*z)/12}" />
-  	</macro>
-  	<macro name="cylinder_inertia" params="m r h">
-	    <inertia  ixx="${m*(3*r*r+h*h)/12}" ixy = "0" ixz = "0"
-	              iyy="${m*(3*r*r+h*h)/12}" iyz = "0"
-	              izz="${m*r*r/2}" />
-	</macro>
-	<link name="base_footprint">  <!-- used because KDL doesnt not support a root link with an inertia -->
-   		<visual>
-			<geometry>
-      				<box size="0.001 0.001 0.001"/>
-     			</geometry>
-			<origin rpy="0 0 0" xyz="0 0 0"/>
-   		</visual>
- 	</link>
-	<gazebo reference="base_footprint">
-		<material>Gazebo/Green</material>
-		<turnGravityOff>false</turnGravityOff>
-	</gazebo>
-	<joint name="base_footprint_joint" type="fixed">
-		<origin xyz="0 0 0" />
-		<parent link="base_footprint" />
-		<child link="base_link" />
-	</joint>
-	<link name="base_link">
-	   		<visual>
-				<geometry>
-	      				<!--<box size="${base_x_size} ${base_y_size} ${base_z_size}"/> -->
-					<box size="0.001 0.001 0.001"/>
-	     			</geometry>
-				<origin rpy="0 0 0" xyz="0 0 0"/>
-				<material name="white">
-					<color rgba="1 1 1 1"/>
-				</material>
-	   		</visual>
-			<collision>
-				<origin rpy="0 0 0" xyz="0 0 ${radius_wheel}"/>
-				<geometry>
-	       				<box size="${base_x_size} ${base_y_size} ${base_z_size}"/>
-				</geometry>
-			</collision>
-			<inertial>
-	      		<mass value="1" />
-	      			<origin xyz="0 0 0" />
-	      			<!--The 3x3 rotational inertia matrix. -->
-	      			<box_inertia  m="1" x="1" y="1" z="1"/>
-	    		</inertial>
-	 	</link>
-	<link name ="chassis"> <!--The mesh of the car -->
-		<visual>
-				<geometry>
-	      				<mesh filename="package://car_description/meshes/whole_car.stl" scale ="0.001 0.001 0.001"/>
-	     			</geometry>
-				<origin rpy="0 0 0" xyz="0 0 0"/>
-	   		</visual>
-			<collision>
-				<origin rpy="0 0 0" xyz="0 0 ${radius_wheel}"/>
-				<geometry>
-	       				<box size="0.001 0.001 0.001"/>
-				</geometry>
-			</collision>
-			<inertial>
-	      		<mass value="1" />
-	      			<origin xyz="0 0 0" />
-	      			<!--The 3x3 rotational inertia matrix. -->
-	      			<box_inertia  m="1" x="1" y="1" z="1"/>
-	    		</inertial>
-	</link>
-	 <link name="wheel_br">
-   		        <visual>
-     			        <geometry>
-       				  <!-- <cylinder length="${length_wheel}" radius="${radius_wheel}"/> -->
-					<mesh filename="package://car_description/meshes/wheel.stl" />
-     			        </geometry>
-			      <!--  <origin rpy="1.5707 0 0" xyz="0 0 0"/> -->
-				<origin rpy="0 0 0" xyz="0 0 0"/>
-   			        <material name="black"/>
-   		        </visual>
-		        <collision>
-				<origin rpy="1.5707 0 0" xyz="0 0 0"/>
-			        <geometry>
-       				        <cylinder length="${length_wheel}" radius="${radius_wheel}"/>
-			        </geometry>
-		        </collision>
-		<inertial>
-                <mass value="${wheel_mass}" />
-                        <origin xyz="0 0 0" />
-                        <cylinder_inertia  m="${wheel_mass}" r="${radius_wheel}" h="${length_wheel}" />
-                </inertial>
- 	</link>
- 	<link name="wheel_bl">
-   		        <visual>
-     			        <geometry>
-       				  <!-- <cylinder length="${length_wheel}" radius="${radius_wheel}"/> -->
-					<mesh filename="package://car_description/meshes/wheel.stl" />
-     			        </geometry>
-			        <!--  <origin rpy="1.5707 0 0" xyz="0 0 0"/> -->
-				<origin rpy="0 0 0" xyz="0 0 0"/>
-   			        <material name="black"/>
-   		        </visual>
-		        <collision>
-				<origin rpy="1.5707 0 0" xyz="0 0 0"/>
-			        <geometry>
-       				        <cylinder length="${length_wheel}" radius="${radius_wheel}"/>
-			        </geometry>
-		        </collision>
-		<inertial>
-                <mass value="${wheel_mass}" />
-                        <origin xyz="0 0 0" />
-                        <cylinder_inertia  m="${wheel_mass}" r="${radius_wheel}" h="${length_wheel}" />
-                </inertial>
- 	</link>
-	 <link name="wheel_fr">
-   		        <visual>
-     			        <geometry>
-       				   <!-- <cylinder length="${length_wheel}" radius="${radius_wheel}"/> -->
-					<mesh filename="package://car_description/meshes/wheel.stl" />
-     			        </geometry>
-			       <!--  <origin rpy="1.5707 0 0" xyz="0 0 0"/> -->
-				<origin rpy="0 0 0" xyz="0 0 0"/>
-   			        <material name="black"/>
-   		        </visual>
-		        <collision>
-				<origin rpy="1.5707 0 0" xyz="0 0 0"/>
-			        <geometry>
-       				        <cylinder length="${length_wheel}" radius="${radius_wheel}"/>
-			        </geometry>
-		        </collision>
-		<inertial>
-                <mass value="${wheel_mass}" />
-                        <origin xyz="0 0 0" />
-                        <cylinder_inertia  m="${wheel_mass}" r="${radius_wheel}" h="${length_wheel}" />
-                </inertial>
- 	</link>
-         <link name="wheel_fl">
-   		        <visual>
-     			        <geometry>
-       				        <!-- <cylinder length="${length_wheel}" radius="${radius_wheel}"/> -->
-					<mesh filename="package://car_description/meshes/wheel.stl" />
-     			        </geometry>
-			       <!--  <origin rpy="1.5707 0 0" xyz="0 0 0"/> -->
-				<origin rpy="0 0 0" xyz="0 0 0"/>
-   			        <material name="black"/>
-   		        </visual>
-		        <collision>
-				<origin rpy="1.5707 0 0" xyz="0 0 0"/>
-			        <geometry>
-       				        <cylinder length="${length_wheel}" radius="${radius_wheel}"/>
-			        </geometry>
-		        </collision>
-		<inertial>
-                <mass value="${wheel_mass}" />
-                        <origin xyz="0 0 0" />
-                        <cylinder_inertia  m="${wheel_mass}" r="${radius_wheel}" h="${length_wheel}" />
-                </inertial>
- 	</link>
-	<xacro:include filename="$(find car_description)/urdf/robot.gazebo" />
-	<link name="turner_right">
-		   		<visual>
-					<geometry>
-		      				<box size="0.000005 0.000005 .000005"/>
-		     			</geometry>
-					<origin rpy="0 0 0" xyz="0 0 0"/>
-					<material name="red">
-						<color rgba="1 0 0 1"/>
-					</material>
-		   		</visual>
-				<collision>
-					<geometry>
-		       				<box size="0.05 0.05 .005"/>
-					</geometry>
-				</collision>
-				<inertial>
-		      		<mass value="1" />
-		      			<origin xyz="0 0 0" />
-		      			<!--The 3x3 rotational inertia matrix. -->
-		      			<box_inertia  m="1" x="0.05" y="0.4" z="0.05"/>
-		    		</inertial>
-		 	</link>
-	<link name="turner_left">
-			   		<visual>
-						<geometry>
-			      				<box size="0.00005 0.00005 .000005"/>
-			     			</geometry>
-						<origin rpy="0 0 0" xyz="0 0 0"/>
-						<material name="red">
-							<color rgba="1 0 0 1"/>
-						</material>
-			   		</visual>
-					<collision>
-						<geometry>
-			       				<box size="0.05 0.05 .005"/>
-						</geometry>
-					</collision>
-					<inertial>
-			      		<mass value="1" />
-			      			<origin xyz="0 0 0" />
-			      			<!--The 3x3 rotational inertia matrix. -->
-			      			<box_inertia  m="1" x="0.0000005" y="0.0000005" z="0.0000005"/>
-			    		</inertial>
-			 	</link>
- <joint name="Turner_right_position_joint" type="revolute">
- <limit effort="1" velocity="1" lower="-0.4" upper="0.4"/>
-   <parent link="base_link"/>
-   <axis xyz="0 0 1" />
-   <child link="turner_right"/>
-   <origin rpy="0 0 0" xyz="${x_offset} ${y_offset * 0.75} 0"/>
- </joint>
- <joint name="Turner_left_position_joint" type="revolute">
- <limit effort="1" velocity="1" lower="-0.4" upper="0.4"/>
-   <parent link="base_link"/>
-   <axis xyz="0 0 1" />
-   <child link="turner_left"/>
-   <origin rpy="0 0 0" xyz="${x_offset} -${y_offset * 0.75} 0"/>
- </joint>
- <joint name="BackWheel_right_joint" type="continuous">
-   <parent link="base_link"/>
-   <axis xyz="0 1 0" />
-   <child link="wheel_br"/>
-   <origin rpy="0 0 0" xyz="-${x_offset} ${y_offset} 0"/>
- </joint>
- <joint name="BackWheel_left_joint" type="continuous">
-   <parent link="base_link"/>
-   <axis xyz="0 1 0" />
-   <child link="wheel_bl"/>
-   <origin rpy="0 0 0" xyz="-${x_offset} -${y_offset} 0"/>
- </joint>
-<!-- non controllable joints -->
- <joint name="base_to_chassis" type="fixed">
-   <parent link="base_link"/>
-   <axis xyz="0 0 1" />
-   <child link="chassis"/>
-   <origin rpy="0 0 0" xyz="0.8 0 -0.1"/>
- </joint>
- <joint name="Front_right_wheel_joint" type="continuous">
-   <parent link="turner_right"/>
-   <axis xyz="0 1 0" />
-   <child link="wheel_fr"/>
-   <origin rpy="0 0 0" xyz="0 0 0"/>
- </joint>
- <joint name="Front_left_wheel_joint" type="continuous">
-   <parent link="turner_left"/>
-   <axis xyz="0 1 0" />
-   <child link="wheel_fl"/>
-   <origin rpy="0 0 0" xyz="0 0 0"/>
- </joint>
- <!-- transmission -->
+<robot  xmlns:xacro="http://www.ros.org/wiki/xacro"
+        xmlns:sensor="http://playerstage.sourceforge.net/gazebo/xmlschema/#sensor"
+        xmlns:controller="http://playerstage.sourceforge.net/gazebo/xmlschema/#controller"
+        xmlns:interface="http://playerstage.sourceforge.net/gazebo/xmlschema/#interface"
+  name="robot1_xacro">
+  <!-- Car properties !!! Y is forward-->
+  <xacro:property name="base_mass" value="20" /> <!-- in kg-->
+  <xacro:property name="base_x_size" value="2.130" />   <!-- x is mhkos forward -->
+  <xacro:property name="base_y_size" value="0.8935" />   <!-- y is platos -->
+  <xacro:property name="base_z_size" value="0.1" /><!-- z is ipsos -->
+  <!-- Wheels -->
+  <xacro:property name="wheel_mass" value="2" /> <!-- in kg-->
+  <xacro:property name="length_wheel" value="0.190" />
+  <xacro:property name="radius_wheel" value="0.261" />
+  <!-- OFFSETS -->
+  <xacro:property name="x_offset" value="0.7625" /> <!-- metaksonio -->
+  <xacro:property name="y_offset" value="0.5652" /> <!-- metatroxio -->
+  <xacro:property name="z_offset" value="${radius_wheel - 0.0001}" /> <!-- diafora ipsous chassis me rodes -->
+  <macro name="box_inertia" params="m x y z">
+    <inertia  ixx="${m*(y*y+z*z)/12}" ixy = "0" ixz = "0"
+              iyy="${m*(x*x+z*z)/12}" iyz = "0"
+              izz="${m*(x*x+z*z)/12}" />
+  </macro>
+  <macro name="cylinder_inertia" params="m r h">
+    <inertia  ixx="${m*(3*r*r+h*h)/12}" ixy = "0" ixz = "0"
+              iyy="${m*(3*r*r+h*h)/12}" iyz = "0"
+              izz="${m*r*r/2}" />
+  </macro>
+  <link name="base_footprint">  <!-- used because KDL doesnt not support a root link with an inertia -->
+    <visual>
+      <geometry>
+        <box size="0.001 0.001 0.001"/>
+      </geometry>
+      <origin rpy="0 0 0" xyz="0 0 0"/>
+    </visual>
+  </link>
+  <gazebo reference="base_footprint">
+    <material>Gazebo/Green</material>
+    <turnGravityOff>false</turnGravityOff>
+  </gazebo>
+  <joint name="base_footprint_joint" type="fixed">
+    <origin xyz="0 0 0" />
+    <parent link="base_footprint" />
+    <child link="base_link" />
+  </joint>
+  <link name="base_link">
+    <visual>
+      <geometry>
+        <!--<box size="${base_x_size} ${base_y_size} ${base_z_size}"/> -->
+        <box size="0.001 0.001 0.001"/>
+      </geometry>
+      <origin rpy="0 0 0" xyz="0 0 0"/>
+      <material name="white">
+        <color rgba="1 1 1 1"/>
+      </material>
+    </visual>
+    <collision>
+      <origin rpy="0 0 0" xyz="0 0 ${radius_wheel}"/>
+      <geometry>
+        <box size="${base_x_size} ${base_y_size} ${base_z_size}"/>
+      </geometry>
+    </collision>
+    <inertial>
+      <mass value="1" />
+      <origin xyz="0 0 0" />
+      <!--The 3x3 rotational inertia matrix. -->
+      <box_inertia  m="1" x="1" y="1" z="1"/>
+    </inertial>
+  </link>
+  <link name ="chassis"> <!--The mesh of the car -->
+    <visual>
+      <geometry>
+        <mesh filename="package://car_description/meshes/whole_car.stl" scale ="0.001 0.001 0.001"/>
+      </geometry>
+      <origin rpy="0 0 0" xyz="0 0 0"/>
+    </visual>
+    <collision>
+      <origin rpy="0 0 0" xyz="0 0 ${radius_wheel}"/>
+      <geometry>
+        <box size="0.001 0.001 0.001"/>
+      </geometry>
+    </collision>
+    <inertial>
+      <mass value="1" />
+      <origin xyz="0 0 0" />
+      <!--The 3x3 rotational inertia matrix. -->
+      <box_inertia  m="1" x="1" y="1" z="1"/>
+    </inertial>
+  </link>
+  <link name="wheel_br">
+    <visual>
+      <geometry>
+        <!-- <cylinder length="${length_wheel}" radius="${radius_wheel}"/> -->
+        <mesh filename="package://car_description/meshes/wheel.stl" />
+      </geometry>
+      <!--  <origin rpy="1.5707 0 0" xyz="0 0 0"/> -->
+      <origin rpy="0 0 0" xyz="0 0 0"/>
+      <material name="black"/>
+    </visual>
+    <collision>
+      <origin rpy="1.5707 0 0" xyz="0 0 0"/>
+        <geometry>
+          <cylinder length="${length_wheel}" radius="${radius_wheel}"/>
+        </geometry>
+      </collision>
+    <inertial>
+      <mass value="${wheel_mass}" />
+      <origin xyz="0 0 0" />
+      <cylinder_inertia  m="${wheel_mass}" r="${radius_wheel}" h="${length_wheel}" />
+    </inertial>
+  </link>
+  <link name="wheel_bl">
+    <visual>
+      <geometry>
+        <!-- <cylinder length="${length_wheel}" radius="${radius_wheel}"/> -->
+        <mesh filename="package://car_description/meshes/wheel.stl" />
+      </geometry>
+      <!--  <origin rpy="1.5707 0 0" xyz="0 0 0"/> -->
+      <origin rpy="0 0 0" xyz="0 0 0"/>
+      <material name="black"/>
+    </visual>
+    <collision>
+      <origin rpy="1.5707 0 0" xyz="0 0 0"/>
+      <geometry>
+        <cylinder length="${length_wheel}" radius="${radius_wheel}"/>
+      </geometry>
+    </collision>
+    <inertial>
+      <mass value="${wheel_mass}" />
+      <origin xyz="0 0 0" />
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