Commit message: removed base_link collision for testing the car's turning car.xacro

File: 3_control/car_description_vel/urdf/car.xacro (robot description, xacro)
@@ -59,5 +59,6 @@
       <origin rpy="0 0 0" xyz="0 0 ${radius_wheel}"/>
       <geometry>
-        <box size="${base_x_size} ${base_y_size} ${base_z_size}"/>
+        <box size="0.001 0.001 0.001"/> <!-- removed collision for testing -->
+        <!-- <box size="${base_x_size} ${base_y_size} ${base_z_size}"/> -->
       </geometry>
     </collision>
