Commit message: Fix lidar and spawn point

File: 3_control/eufs_description/robots/ads-dv.urdf.xacro (robot description, xacro)
@@ -44,68 +44,12 @@
   STEREO CAM: -0.110 0.0 0.800 -->
   <xacro:sensor_imu parent="base_link" prefix="imu">
-      <origin xyz="-0.0 0.0 0.0" rpy="0 0 0"/>
+    <origin xyz="-0.0 0.0 0.0" rpy="0 0 0"/>
   </xacro:sensor_imu>
   <xacro:sensor_gps  parent="base_link" prefix="gps">
-      <origin xyz="0.0 0.0 0.4" rpy="0 0 0"/>
+    <origin xyz="0.0 0.0 0.4" rpy="0 0 0"/>
   </xacro:sensor_gps>
-  <!-- Hokuyo joint -->
-  <joint name="hokuyo_joint" type="fixed">
-    <origin xyz="1.58 0.0 -0.1" rpy="0 0 0"/>
-    <parent link="base_link"/>
-    <axis xyz="0 1 0" />
-    <child link="hokuyo_link"/>
-  </joint>
-  <!-- Hokuyo Laser -->
-  <link name="hokuyo_link">
-<!--      <collision>-->
-<!--        <origin xyz="0 0 0" rpy="0 0 0"/>-->
-<!--        <geometry>-->
-<!--          <box size="0.01 -0.05 0.06"/>-->
-<!--        </geometry>-->
-<!--      </collision>-->
-    <visual>
-      <origin xyz="0 -0.05 0.06" rpy="0 0 0"/>
-      <geometry>
-        <mesh filename="package://robot/meshes/hokuyo.dae"/>
-      </geometry>
-    </visual>
-    <inertial>
-      <mass value="1e-5" />
-      <origin xyz="0 0 0" rpy="0 0 0"/>
-      <inertia ixx="1e-6" ixy="0" ixz="0" iyy="1e-6" iyz="0" izz="1e-6" />
-    </inertial>
-  </link>
-  <gazebo reference="hokuyo_link">
-    <sensor type="ray" name="head_hokuyo_sensor">
-      <pose>0 0 0 0 0 0</pose>
-      <visualize>false</visualize>
-      <update_rate>40</update_rate>
-      <ray>
-        <scan>
-          <horizontal>
-            <samples>720</samples>
-            <resolution>1</resolution>
-            <min_angle>-1.570796</min_angle>
-            <max_angle>1.570796</max_angle>
-          </horizontal>
-        </scan>
-        <range>
-          <min>0.10</min>
-          <max>30.0</max>
-          <resolution>0.01</resolution>
-        </range>
-        <noise>
-          <type>gaussian</type>
-          <mean>0.0</mean>
-          <stddev>0.01</stddev>
-        </noise>
-      </ray>
-      <plugin name="gazebo_ros_head_hokuyo_controller" filename="libgazebo_ros_laser.so">
-        <topicName>scan</topicName>
-        <frameName>hokuyo_link</frameName>
-<!--        <robotNamespace>/robot</robotNamespace>-->
-      </plugin>
-    </sensor>
-  </gazebo>
+  <xacro:sensor_hokuyo_utm30lx  parent="base_link" prefix="lidar" >
+    <origin xyz="1.700 0.0 -0.080" rpy="0 0 0"/>
+  </xacro:sensor_hokuyo_utm30lx>
   <!-- <xacro:VLP-16  parent="base_link" name="velodyne" topic="/velodyne_points" hz="10">
       <origin xyz="1.700 0.0 -0.150" rpy="0 -0.0174533 0"/>
@@ -115,5 +59,5 @@
 <!--    </xacro:VLP-16R>-->
   <xacro:zed_camera parent="base_link" prefix="zed">
-      <origin xyz="0.1 0.0 0.52" rpy="0 0 0"/>
+    <origin xyz="0.1 0.0 0.52" rpy="0 0 0"/>
   </xacro:zed_camera>
   <!-- EXTRA SENSORS FROM THE ROBOTNIK SENSORS LIBRARY -->

File: 3_control/eufs_description/sensors/hokuyo_utm30lx.urdf.xacro (robot description, xacro)
@@ -1,16 +1,15 @@
 <?xml version="1.0"?>
-<robot name="sensor_hokuyo" xmlns:xacro="http://www.ros.org/wiki/xacro">
-  <xacro:macro name="sensor_hokuyo" >
-    <joint name="hokuyo_joint" type="fixed">
+<robot name="sensor_hokuyo_utm30lx" xmlns:xacro="http://www.ros.org/wiki/xacro">
+  <xacro:macro name="sensor_hokuyo_utm30lx" params="prefix:=-eufs parent:=base_link prefix_topic:=eufs *origin min_angle:=-1.57 max_angle:=1.57">
+    <joint name="${prefix}_base_joint" type="fixed">
       <!-- FRONT MOUNT  -->
       <!-- origin xyz="0.29 0 0.1" -->
       <!-- TOP MOUNT -->
       <!-- origin xyz="0.0 0.0 0.325"-->
-<!--      <xacro:insert_block name="origin"/>-->
-      <origin xyz="0.29 0 0.1" rpy="0 0 0"/>
-      <parent link="base_link"/>
-      <child link="hokuyo_link"/>
+      <xacro:insert_block name="origin"/>
+      <parent link="${parent}"/>
+      <child link="${prefix}_base_link"/>
     </joint>
-    <link name="hokuyo_link">
+    <link name="${prefix}_base_link">
       <visual>
         <origin rpy="0 0 0" xyz="0 0 0"/>
@@ -25,19 +24,19 @@
       </inertial>
     </link>
-<!--    <link name="${prefix}_link"/>-->
-<!--    <joint name="${prefix}_joint" type="fixed">-->
-<!--      <parent link="${prefix}_base_link"/>-->
-<!--      <child link="${prefix}_link"/>-->
-<!--      <origin rpy="0 0 0" xyz="0.00 0 0.055"/>-->
-<!--    </joint>-->
+    <link name="${prefix}_link"/>
+    <joint name="${prefix}_joint" type="fixed">
+      <parent link="${prefix}_base_link"/>
+      <child link="${prefix}_link"/>
+      <origin rpy="0 0 0" xyz="0.00 0 0.055"/>
+    </joint>
     <!-- Hokuyo sensor for simulation -->
-<!--    <sensor_hokuyo_utm_gazebo/>-->
+    <sensor_hokuyo_utm_gazebo/>
   </xacro:macro>
-  <xacro:macro name="sensor_hokuyo">
-    <gazebo reference="hokuyo_link">
-      <sensor name="hokuyo_sensor" type="ray">
+  <xacro:macro name="sensor_hokuyo_utm_gazebo">
+    <gazebo reference="${prefix}_link">
+      <sensor name="${prefix}_sensor" type="ray">
         <pose>0 0 0 0 0 0</pose>
-        <visualize>true</visualize>
-        <update_rate>30</update_rate>
+        <visualize>false</visualize>
+        <update_rate>40</update_rate>
         <ray>
           <scan>
@@ -45,11 +44,11 @@
               <samples>1081</samples>
               <resolution>1</resolution>
-              <min_angle>-1.570796</min_angle>
-              <max_angle>1.570796</max_angle>
+              <min_angle>${min_angle}</min_angle>
+              <max_angle>${max_angle}</max_angle>
             </horizontal>
           </scan>
           <range>
             <min>0.10</min>
-            <max>30.0</max>
+            <max>15.0</max>
             <resolution>0.01</resolution>
           </range>
@@ -60,7 +59,7 @@
           </noise>
         </ray>
-        <plugin filename="libgazebo_ros_laser.so" name="hokuyo_controller">
+        <plugin filename="libgazebo_ros_laser.so" name="${prefix}_controller">
           <topicName>scan</topicName>
-          <frameName>hokuyo_link</frameName>
+          <frameName>/${prefix}_link</frameName>
         </plugin>
       </sensor>

Commit message: Remove useless xacros, comment p3d, gps

File: 3_control/eufs_description/robots/ads-dv.urdf.xacro (robot description, xacro)
@@ -46,7 +46,7 @@
     <origin xyz="-0.0 0.0 0.0" rpy="0 0 0"/>
   </xacro:sensor_imu>
-  <xacro:sensor_gps  parent="base_link" prefix="gps">
-    <origin xyz="0.0 0.0 0.4" rpy="0 0 0"/>
-  </xacro:sensor_gps>
+<!--  <xacro:sensor_gps  parent="base_link" prefix="gps">-->
+<!--    <origin xyz="0.0 0.0 0.4" rpy="0 0 0"/>-->
+<!--  </xacro:sensor_gps>-->
   <xacro:sensor_hokuyo_utm30lx  parent="base_link" prefix="lidar" >
     <origin xyz="1.700 0.0 -0.080" rpy="0 0 0"/>

File: 3_control/eufs_description/urdf/bases/ads-dv_base.urdf.xacro (robot description, xacro)
@@ -59,22 +59,22 @@
     </collision>
   </link>
-  <link name="odom_ground_truth">
-    <collision>
-      <geometry>
-        <box size="0.1 0.1 0.1"/>
-      </geometry>
-    </collision>
-    <inertial>
-      <mass value="1e-5" />
-      <origin xyz="0 0 0" rpy="0 0 0"/>
-      <inertia ixx="1e-6" ixy="0" ixz="0" iyy="1e-6" iyz="0" izz="1e-6" />
-    </inertial>
-  </link>
-  <joint name="odom_ground_truth_joint" type="fixed">
-    <axis xyz="0 0 0" />
-    <origin xyz="0 0 0" rpy="0 0 0"/>
-    <parent link="base_link"/>
-    <child link="odom_ground_truth"/>
-  </joint>
+<!--  <link name="odom_ground_truth">-->
+<!--    <collision>-->
+<!--      <geometry>-->
+<!--        <box size="0.1 0.1 0.1"/>-->
+<!--      </geometry>-->
+<!--    </collision>-->
+<!--    <inertial>-->
+<!--      <mass value="1e-5" />-->
+<!--      <origin xyz="0 0 0" rpy="0 0 0"/>-->
+<!--      <inertia ixx="1e-6" ixy="0" ixz="0" iyy="1e-6" iyz="0" izz="1e-6" />-->
+<!--    </inertial>-->
+<!--  </link>-->
+<!--  <joint name="odom_ground_truth_joint" type="fixed">-->
+<!--    <axis xyz="0 0 0" />-->
+<!--    <origin xyz="0 0 0" rpy="0 0 0"/>-->
+<!--    <parent link="base_link"/>-->
+<!--    <child link="odom_ground_truth"/>-->
+<!--  </joint>-->
   </xacro:macro>
 </robot>

File: 3_control/eufs_description/urdf/bases/eufs_base.gazebo.xacro (robot description, xacro)
@@ -13,17 +13,17 @@
     </gazebo>
 	</xacro:macro>
-  <gazebo>
-    <plugin name="p3d_base_controller" filename="libgazebo_ros_p3d.so">
-        <alwaysOn>true</alwaysOn>
-        <updateRate>200.0</updateRate>
-        <bodyName>odom_ground_truth</bodyName>
-        <topicName>ground_truth/state_raw</topicName>
-        <gaussianNoise>0.00</gaussianNoise>
-        <frameName>world</frameName>
-        <!-- origin is at spawn location -->
-        <xyzOffset>43.0 -40 0</xyzOffset>
-        <rpyOffset>0 0 0</rpyOffset>
-    </plugin>
-  </gazebo>
+<!--  <gazebo>	-->
+<!--    <plugin name="p3d_base_controller" filename="libgazebo_ros_p3d.so">-->
+<!--        <alwaysOn>true</alwaysOn>-->
+<!--        <updateRate>200.0</updateRate>-->
+<!--        <bodyName>odom_ground_truth</bodyName>-->
+<!--        <topicName>ground_truth/state_raw</topicName>-->
+<!--        <gaussianNoise>0.00</gaussianNoise>-->
+<!--        <frameName>world</frameName>-->
+<!--        <!-- origin is at spawn location -->-->
+<!--        <xyzOffset>43.0 -40 0</xyzOffset>-->
+<!--        <rpyOffset>0 0 0</rpyOffset>-->
+<!--    </plugin>-->
+<!--  </gazebo>-->
   <!-- No Ackermann steering plugin -->
   <gazebo reference="base_footprint">

Commit message: Add YOLO

File: 3_control/eufs_description/robots/ads-dv.urdf.xacro (robot description, xacro)
@@ -46,7 +46,7 @@
     <origin xyz="-0.0 0.0 0.0" rpy="0 0 0"/>
   </xacro:sensor_imu>
-<!--  <xacro:sensor_gps  parent="base_link" prefix="gps">-->
-<!--    <origin xyz="0.0 0.0 0.4" rpy="0 0 0"/>-->
-<!--  </xacro:sensor_gps>-->
+  <xacro:sensor_gps  parent="base_link" prefix="gps">
+    <origin xyz="0.0 0.0 0.4" rpy="0 0 0"/>
+  </xacro:sensor_gps>
   <xacro:sensor_hokuyo_utm30lx  parent="base_link" prefix="lidar" >
     <origin xyz="1.700 0.0 -0.080" rpy="0 0 0"/>
@@ -58,7 +58,7 @@
 <!--        <origin xyz="1.58 0.0 -0.1" rpy="0 ${1*M_PI/180.0} 0"/>-->
 <!--    </xacro:VLP-16R>-->
-  <xacro:zed_camera parent="base_link" prefix="zed">
-    <origin xyz="0.1 0.0 0.52" rpy="0 0 0"/>
-  </xacro:zed_camera>
+  <xacro:sensor_kinect parent="base_link" prefix="kinect">
+      <origin xyz="0.1 0.0 0.52" rpy="0 0 0"/>
+  </xacro:sensor_kinect>
   <!-- EXTRA SENSORS FROM THE ROBOTNIK SENSORS LIBRARY -->
 <!--
@@ -75,7 +75,7 @@
       <origin xyz="0.3 0.0 0.3" rpy="0 0 0"/>
   </xacro:sensor_asus_xtion_pro>
-  <xacro:sensor_kinect parent="base_link" prefix="kinect">
-      <origin xyz="0.0 0.0 0.45" rpy="0 0 0"/>
-  </xacro:sensor_kinect>
+  <xacro:zed_camera parent="base_link" prefix="zed">
+    <origin xyz="0.1 0.0 0.52" rpy="0 0 0"/>
+  </xacro:zed_camera>
   <xacro:BB2-08S2C-60  prefix="bee" frame="bee" name="bee"/>
   <xacro:sensor_fotonic name="fotonic" parent="base_link">

Commit message: Use zed camera with yolo

File: 3_control/eufs_description/robots/ads-dv.urdf.xacro (robot description, xacro)
@@ -58,7 +58,7 @@
 <!--        <origin xyz="1.58 0.0 -0.1" rpy="0 ${1*M_PI/180.0} 0"/>-->
 <!--    </xacro:VLP-16R>-->
-  <xacro:sensor_kinect parent="base_link" prefix="kinect">
-      <origin xyz="0.1 0.0 0.52" rpy="0 0 0"/>
-  </xacro:sensor_kinect>
+  <xacro:zed_camera parent="base_link" prefix="zed">
+    <origin xyz="0.1 0.0 0.52" rpy="0 0 0"/>
+  </xacro:zed_camera>
   <!-- EXTRA SENSORS FROM THE ROBOTNIK SENSORS LIBRARY -->
 <!--
@@ -75,7 +75,7 @@
       <origin xyz="0.3 0.0 0.3" rpy="0 0 0"/>
   </xacro:sensor_asus_xtion_pro>
-  <xacro:zed_camera parent="base_link" prefix="zed">
-    <origin xyz="0.1 0.0 0.52" rpy="0 0 0"/>
-  </xacro:zed_camera>
+  <xacro:sensor_kinect parent="base_link" prefix="kinect">
+      <origin xyz="0.1 0.0 0.52" rpy="0 0 0"/>
+  </xacro:sensor_kinect>
   <xacro:BB2-08S2C-60  prefix="bee" frame="bee" name="bee"/>
   <xacro:sensor_fotonic name="fotonic" parent="base_link">
